Commit message: Init

File: src/example_robot_model/urdf/my_robotic_arm.urdf (robot description, URDF)
Before this commit: robot exmaple_robot_model, 9 links, 8 joints
Links:
- link end: geometry collision mesh filename=package://example_robot_model/meshes/end.STL; visual mesh filename=package://example_robot_model/meshes/end.STL
- link r1: geometry collision mesh filename=package://example_robot_model/meshes/r1.STL; visual mesh filename=package://example_robot_model/meshes/r1.STL
- link r2: geometry collision mesh filename=package://example_robot_model/meshes/r2.STL; visual mesh filename=package://example_robot_model/meshes/r2.STL
- link r3: geometry collision mesh filename=package://example_robot_model/meshes/r3.STL; visual mesh filename=package://example_robot_model/meshes/r3.STL
- link r4: geometry collision mesh filename=package://example_robot_model/meshes/r4.STL; visual mesh filename=package://example_robot_model/meshes/r4.STL
- link r5: geometry collision mesh filename=package://example_robot_model/meshes/r5.STL; visual mesh filename=package://example_robot_model/meshes/r5.STL
- link r6: geometry collision mesh filename=package://example_robot_model/meshes/r6.STL; visual mesh filename=package://example_robot_model/meshes/r6.STL
- link r7: geometry collision mesh filename=package://example_robot_model/meshes/r7.STL; visual mesh filename=package://example_robot_model/meshes/r7.STL
- link robot_base: geometry collision mesh filename=package://example_robot_model/meshes/base.STL; visual mesh filename=package://example_robot_model/meshes/base.STL
