Commit message: 秒了，没报错

File: src/engineering_robot/urdf/engineering_robot.urdf (robot description, URDF)
Before this commit: robot engineering_robot, 8 links, 7 joints
Links:
- link J1_pris: mass 1.0672 -> 0.91288340947747
- link J1_rotate: mass 0.98991 -> 0.989907036021585
- link J2: mass 0.383011983841491 -> 0.47390104289524
- link J3: mass 0.45196060079211 -> 0.451960600792109
- link J4_x: mass 0.245833034470926 -> 0.245833034470928
- link J4_y: mass 0.24583 -> 0.245833034470928
- link J5_end: mass 0.10668 -> 0.106684158826586
- link robot_base: mass 22.186 -> 22.1862077008472
Joints:
- joint J1_pris: limit lower=0 upper=0.4 effort=0 velocity=0.0225 -> lower=-0.4 upper=0 effort=0 velocity=0.0225

Commit message: ok 倒入成功

File: src/engineering_robot/urdf/engineering_robot.urdf (robot description, URDF)
Before this commit: robot engineering_robot, 8 links, 7 joints
Joints:
- removed joint J1_pris
- removed joint J1_rotate
- removed joint J2
- removed joint J3
- removed joint J4_x
- removed joint J4_y
- removed joint J5_end
- added joint J1_pris_: type prismatic, parent robot_base, child J1_pris, origin xyz=-0.046 -0.1815 0.208 rpy=0 0 3.1416, axis 0 0 -1, limit lower=-0.4 upper=0 effort=0 velocity=0.0225
- added joint J1_rotate_: type revolute, parent J1_pris, child J1_rotate, origin xyz=0 0 0 rpy=0 0 0, axis 0 0 -1, limit lower=-3.14 upper=3.14 effort=0 velocity=3.0
- added joint J2_: type revolute, parent J1_rotate, child J2, origin xyz=0.004527 0.21888 0.043 rpy=0 0 -0.020679, axis 0 0 -1, limit lower=-3.14 upper=3.14 effort=0 velocity=3.0
- added joint J3_: type revolute, parent J2, child J3, origin xyz=-0.014396 0.11107 0.059 rpy=0 -0.12124 0.12889, axis 0 -1 0, limit lower=-3.14 upper=3.14 effort=0 velocity=3.0
- added joint J4_x_: type revolute, parent J3, child J4_x, origin xyz=-0.0002 0.18972 -0.085 rpy=0.11366 0 0, axis -1 0 0, limit lower=-3.14 upper=3.14 effort=0 velocity=3.0
- added joint J4_y_: type revolute, parent J4_x, child J4_y, origin xyz=0 0 0 rpy=0 0 0, axis 0 -1 0, limit lower=-10000 upper=10000 effort=0 velocity=3.0
- added joint J5_end_: type fixed, parent J4_y, child J5_end, origin xyz=0 0.1105 0 rpy=0 0 0, axis 0 0 0

File: src/engineering_robot_moveit/config/engineering_robot.ros2_control.xacro (robot description, xacro)
@@ -8,49 +8,49 @@
                 <plugin>mock_components/GenericSystem</plugin>
             </hardware>
-            <joint name="J1_pris">
+            <joint name="J1_pris_">
                 <command_interface name="position"/>
                 <command_interface name="velocity"/>
                 <state_interface name="position">
-                  <param name="initial_value">${initial_positions['J1_pris']}</param>
+                  <param name="initial_value">${initial_positions['J1_pris_']}</param>
                 </state_interface>
                 <state_interface name="velocity"/>
             </joint>
-            <joint name="J1_rotate">
+            <joint name="J1_rotate_">
                 <command_interface name="position"/>
                 <command_interface name="velocity"/>
                 <state_interface name="position">
-                  <param name="initial_value">${initial_positions['J1_rotate']}</param>
+                  <param name="initial_value">${initial_positions['J1_rotate_']}</param>
                 </state_interface>
                 <state_interface name="velocity"/>
             </joint>
-            <joint name="J2">
+            <joint name="J2_">
                 <command_interface name="position"/>
                 <command_interface name="velocity"/>
                 <state_interface name="position">
-                  <param name="initial_value">${initial_positions['J2']}</param>
+                  <param name="initial_value">${initial_positions['J2_']}</param>
                 </state_interface>
                 <state_interface name="velocity"/>
             </joint>
-            <joint name="J3">
+            <joint name="J3_">
                 <command_interface name="position"/>
                 <command_interface name="velocity"/>
                 <state_interface name="position">
-                  <param name="initial_value">${initial_positions['J3']}</param>
+                  <param name="initial_value">${initial_positions['J3_']}</param>
                 </state_interface>
                 <state_interface name="velocity"/>
             </joint>
-            <joint name="J4_x">
+            <joint name="J4_x_">
                 <command_interface name="position"/>
                 <command_interface name="velocity"/>
                 <state_interface name="position">
-                  <param name="initial_value">${initial_positions['J4_x']}</param>
+                  <param name="initial_value">${initial_positions['J4_x_']}</param>
                 </state_interface>
                 <state_interface name="velocity"/>
             </joint>
-            <joint name="J4_y">
+            <joint name="J4_y_">
                 <command_interface name="position"/>
                 <command_interface name="velocity"/>
                 <state_interface name="position">
-                  <param name="initial_value">${initial_positions['J4_y']}</param>
+                  <param name="initial_value">${initial_positions['J4_y_']}</param>
                 </state_interface>
                 <state_interface name="velocity"/>

Commit message: ok，可以跑了，但是启动缓慢 [move_group-3] [WARN] [1745930407.133768576] [moveit_ros.planning_scene_monitor.planning_scene_monitor]: It is likely there are too many vertices in collision geometry

File: src/engineering_robot/urdf/engineering_robot.urdf (robot description, URDF)
Before this commit: robot engineering_robot, 8 links, 7 joints
Joints:
- joint J4_y_: limit lower=-10000 upper=10000 effort=0 velocity=3.0 -> lower=-1.57 upper=1.57 effort=0 velocity=3.0

Commit message: 导入了新的模型，并且修复了代码

File: src/engineering_robot/urdf/engineering_robot.urdf (robot description, URDF)
Before this commit: robot engineering_robot, 8 links, 7 joints
Links:
- removed link J1_pris
- removed link J1_rotate
- removed link J2
- removed link J3
- removed link J4_x
- removed link J4_y
- removed link J5_end
- removed link robot_base
- added link J1_link, mass 1.2292; collision mesh filename=package://engineering_robot/meshes/J1_link.STL; visual mesh filename=package://engineering_robot/meshes/J1_link.STL
- added link J2_link, mass 0.70346; collision mesh filename=package://engineering_robot/meshes/J2_link.STL; visual mesh filename=package://engineering_robot/meshes/J2_link.STL
- added link J3_link, mass 0.82034; collision mesh filename=package://engineering_robot/meshes/J3_link.STL; visual mesh filename=package://engineering_robot/meshes/J3_link.STL
- added link J4_link, mass 1.4198; collision mesh filename=package://engineering_robot/meshes/J4_link.STL; visual mesh filename=package://engineering_robot/meshes/J4_link.STL
- added link J5_x_link, mass 0.042542; collision mesh filename=package://engineering_robot/meshes/J5_x_link.STL; visual mesh filename=package://engineering_robot/meshes/J5_x_link.STL
- added link J5_z_link, mass 0.042542; collision mesh filename=package://engineering_robot/meshes/J5_z_link.STL; visual mesh filename=package://engineering_robot/meshes/J5_z_link.STL
- added link end_link, mass 0.088683; collision mesh filename=package://engineering_robot/meshes/end_link.STL; visual mesh filename=package://engineering_robot/meshes/end_link.STL
- added link robot_base_link, mass 11.763; collision mesh filename=package://engineering_robot/meshes/robot_base_link.STL; visual mesh filename=package://engineering_robot/meshes/robot_base_link.STL
Joints:
- removed joint J1_pris_
- removed joint J1_rotate_
- removed joint J2_
- removed joint J3_
- removed joint J4_x_
- removed joint J4_y_
- removed joint J5_end_
- added joint J1J: type prismatic, parent robot_base_link, child J1_link, origin xyz=0.051 0.398 -0.041 rpy=0 0 0, axis 0 0 -1, limit lower=4 upper=0 effort=0 velocity=0.045
- added joint J2J: type revolute, parent J1_link, child J2_link, origin xyz=0 0 0 rpy=0 0 0, axis 0 0 -1, limit lower=-3.1415926 upper=3.1415926 effort=0 velocity=3.5
- added joint J3J: type revolute, parent J2_link, child J3_link, origin xyz=0.00034388 0.2195 0.066 rpy=0 0 -0.0050473, axis 0 0 -1, limit lower=-3.1415926 upper=3.1415926 effort=0 velocity=3.5
- added joint J4J: type revolute, parent J3_link, child J4_link, origin xyz=0.00046225 0.103 0.0457 rpy=0 0 -0.0044879, axis 0 -1 0, limit lower=-3.1415926 upper=3.1415926 effort=0 velocity=3.5
- added joint J5_xJ: type revolute, parent J4_link, child J5_x_link, origin xyz=-0.00049488 0.19759 -0.08712 rpy=0.0060187 0.0056803 0, axis 1 0 0, limit lower=-3.1415926 upper=3.1415926 effort=0 velocity=3.5
- added joint J5_zJ: type revolute, parent J5_x_link, child J5_z_link, origin xyz=0 0 0 rpy=0 0 0, axis 0 0 -1, limit lower=-3.1415926 upper=3.1415926 effort=0 velocity=3.5
- added joint end: type fixed, parent J5_z_link, child end_link, origin xyz=0 0 -0.137 rpy=-3.1416 0 0, axis 0 0 0

Commit message: 适配新模型

File: src/engineering_robot/urdf/engineering_robot.urdf (robot description, URDF)
Before this commit: robot engineering_robot, 8 links, 7 joints
Links:
- link J1_link: mass 1.2292 -> 1.22922743338823
- link J2_link: mass 0.70346 -> 0.70345662801813
- link J3_link: mass 0.82034 -> 0.820340126206514
- link J4_link: mass 1.4198 -> 1.4197918033911
- link J5_x_link: mass 0.042542 -> 0.0425415484567542
- link J5_z_link: mass 0.042542 -> 0.0425415484567542
- link end_link: mass 0.088683 -> 0.0886825393828937
- link robot_base_link: mass 11.763 -> 11.7630413668717
Joints:
- joint J1J: limit lower=4 upper=0 effort=0 velocity=0.045 -> lower=-0.46 upper=0 effort=0 velocity=0.045
- joint J2J: limit lower=-3.1415926 upper=3.1415926 effort=0 velocity=3.5 -> lower=-3.1416 upper=3.1416 effort=0 velocity=3.5
- joint J3J: limit lower=-3.1415926 upper=3.1415926 effort=0 velocity=3.5 -> lower=-3.1416 upper=3.1416 effort=0 velocity=3.5
- joint J4J: limit lower=-3.1415926 upper=3.1415926 effort=0 velocity=3.5 -> lower=-3.1416 upper=3.1416 effort=0 velocity=3.5
- joint J5_xJ: limit lower=-3.1415926 upper=3.1415926 effort=0 velocity=3.5 -> lower=-3.1416 upper=3.1416 effort=0 velocity=3.5
- joint J5_zJ: limit lower=-3.1415926 upper=3.1415926 effort=0 velocity=3.5 -> lower=-3.1416 upper=3.1416 effort=0 velocity=3.5

File: src/engineering_robot_moveit/config/engineering_robot.ros2_control.xacro (robot description, xacro)
@@ -6,52 +6,52 @@
             <hardware>
                 <!-- By default, set up controllers for simulation. This won't work on real hardware -->
+                <plugin>Engineering_robot_RM2025_Pnx/ERHardwareInterface</plugin>
                 <!-- <plugin>mock_components/GenericSystem</plugin> -->
-                <plugin>Engineering_robot_RM2025_Pnx/ERHardwareInterface</plugin>
             </hardware>
-            <joint name="J1_pris_">
+            <joint name="J1J">
                 <command_interface name="position"/>
                 <command_interface name="velocity"/>
                 <state_interface name="position">
-                  <param name="initial_value">${initial_positions['J1_pris_']}</param>
+                  <param name="initial_value">${initial_positions['J1J']}</param>
                 </state_interface>
                 <state_interface name="velocity"/>
             </joint>
-            <joint name="J1_rotate_">
+            <joint name="J2J">
                 <command_interface name="position"/>
                 <command_interface name="velocity"/>
                 <state_interface name="position">
-                  <param name="initial_value">${initial_positions['J1_rotate_']}</param>
+                  <param name="initial_value">${initial_positions['J2J']}</param>
                 </state_interface>
                 <state_interface name="velocity"/>
             </joint>
-            <joint name="J2_">
+            <joint name="J3J">
                 <command_interface name="position"/>
                 <command_interface name="velocity"/>
                 <state_interface name="position">
-                  <param name="initial_value">${initial_positions['J2_']}</param>
+                  <param name="initial_value">${initial_positions['J3J']}</param>
                 </state_interface>
                 <state_interface name="velocity"/>
             </joint>
-            <joint name="J3_">
+            <joint name="J4J">
                 <command_interface name="position"/>
                 <command_interface name="velocity"/>
                 <state_interface name="position">
-                  <param name="initial_value">${initial_positions['J3_']}</param>
+                  <param name="initial_value">${initial_positions['J4J']}</param>
                 </state_interface>
                 <state_interface name="velocity"/>
             </joint>
-            <joint name="J4_x_">
+            <joint name="J5_xJ">
                 <command_interface name="position"/>
                 <command_interface name="velocity"/>
                 <state_interface name="position">
-                  <param name="initial_value">${initial_positions['J4_x_']}</param>
+                  <param name="initial_value">${initial_positions['J5_xJ']}</param>
                 </state_interface>
                 <state_interface name="velocity"/>
             </joint>
-            <joint name="J4_y_">
+            <joint name="J5_zJ">
                 <command_interface name="position"/>
                 <command_interface name="velocity"/>
                 <state_interface name="position">
-                  <param name="initial_value">${initial_positions['J4_y_']}</param>
+                  <param name="initial_value">${initial_positions['J5_zJ']}</param>
                 </state_interface>
                 <state_interface name="velocity"/>

File: src/engineering_robot_moveit/config/engineering_robot.urdf.xacro (robot description, xacro)
@@ -6,4 +6,4 @@
     <!-- Import control_xacro -->
     <xacro:include filename="engineering_robot.ros2_control.xacro" />
-    <xacro:engineering_robot_ros2_control name="Realsystem" initial_positions_file="$(arg initial_positions_file)"/>
+    <xacro:engineering_robot_ros2_control name="Realsysystem" initial_positions_file="$(arg initial_positions_file)"/>
 </robot>

Commit message: 测试后存档

File: src/engineering_robot/urdf/engineering_robot.urdf (robot description, URDF)
Before this commit: robot engineering_robot, 8 links, 7 joints
Joints:
- joint J2J: limit lower=-3.1416 upper=3.1416 effort=0 velocity=3.5 -> lower=-1.844444444444444 upper=1.653 effort=0 velocity=5
- joint J3J: limit lower=-3.1416 upper=3.1416 effort=0 velocity=3.5 -> lower=-3.14 upper=3.14 effort=0 velocity=5
- joint J4J: limit lower=-3.1416 upper=3.1416 effort=0 velocity=3.5 -> lower=-3.1416 upper=3.1416 effort=0 velocity=5
- joint J5_xJ: limit lower=-3.1416 upper=3.1416 effort=0 velocity=3.5 -> lower=-3.1416 upper=3.1416 effort=0 velocity=5
- joint J5_zJ: limit lower=-3.1416 upper=3.1416 effort=0 velocity=3.5 -> lower=-3.1416 upper=3.1416 effort=0 velocity=5

Commit message: add mine link but still have some problem

File: src/engineering_robot/urdf/engineering_robot.urdf (robot description, URDF)
Before this commit: robot engineering_robot, 8 links, 7 joints
Links:
- added link mine_link
Joints:
- added joint mine: type fixed, parent end_link, child mine_link, origin xyz=0 0 0.083 rpy=0 0 0, axis 0 0 0
